Commit message: ik for grasping

File: src/sponana/models/grasping/spot_gripper.urdf (robot description, URDF)
Before this commit: robot spot_gripper, 3 links, 2 joints
Links:
- added link foo
Joints:
- added joint foo_weld: type fixed, parent arm_link_wr1, child foo, origin xyz=0. -0.08 0.0 rpy=0 0 1.57

Commit message: clean up grasping code

File: src/sponana/models/grasping/spot_gripper.urdf (robot description, URDF)
Before this commit: robot spot_gripper, 4 links, 3 joints
Joints:
- joint gripper_weld: origin xyz=0. -0.08 0.0 rpy=0 0 1.57 -> xyz=0. -0.08 0.0 rpy=1.57 0 1.57
